File: DMH_Transistor_VCA_PANEL/DMH_Transistor_VCA_PANEL.kicad_sch (KiCad schematic)
At the start: 19 parts, among them J0 Panel_GND_Solder_Wire_Pad

Commit message: Generated Gerbers
Parts:
- H13, H14, H6, H7: footprint SynthStuff:Pot_Cutout_Tiny_attv -> SynthStuff:Pot_Cutout_Tiny_attv_P110KH1
Changed lines of the file:
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@@
 			)
 		)
-		(property "Footprint" "SynthStuff:Pot_Cutout_Tiny_attv"
+		(property "Footprint" "SynthStuff:Pot_Cutout_Tiny_attv_P110KH1"
 			(at 101.6 179.07 0)
 			(effects
@@
 			)
 		)
-		(property "Footprint" "SynthStuff:Pot_Cutout_Tiny_attv"
+		(property "Footprint" "SynthStuff:Pot_Cutout_Tiny_attv_P110KH1"
 			(at 101.6 102.87 0)
 			(effects
@@
 			)
 		)
-		(property "Footprint" "SynthStuff:Pot_Cutout_Tiny_attv"
+		(property "Footprint" "SynthStuff:Pot_Cutout_Tiny_attv_P110KH1"
 			(at 76.2 102.87 0)
 			(effects
@@
 			)
 		)
-		(property "Footprint" "SynthStuff:Pot_Cutout_Tiny_attv"
+		(property "Footprint" "SynthStuff:Pot_Cutout_Tiny_attv_P110KH1"
 			(at 76.2 179.07 0)
 			(effects
