File: DMH_Transistor_VCA_PCB_Conn/Inputs_and_Outputs.kicad_sch (KiCad schematic)
At the start: 0 parts

Commit message: Pots PCB in progress
Need to add CV input traces to the pin headers
Parts:
- added J0: Conn_01x01, Connector_PinHeader_2.54mm:PinHeader_1x01_P2.54mm_Vertical, symbol Connector_Generic:Conn_01x01
- added J1, J2, J3, J4, J5, J6, J7, J8: TS_Jack_6.35mm_Sw, SynthStuff:CUI_MJ-63052A, symbol SynthStuff:TS_Jack_6.35mm_Sw
- added J200: IDC_02x05, SynthStuff:IDC-Header_2x05_P2.54mm_Vertical_BackBone, symbol SynthStuff:BackBone_Connector_10Pin
- added J50, J60: Conn_01x06, Connector_PinHeader_2.54mm:PinHeader_1x06_P2.54mm_Vertical, symbol Connector_Generic:Conn_01x06
- added R21, R40: 20k, Resistor_THT:R_Axial_DIN0207_L6.3mm_D2.5mm_P7.62mm_Horizontal, symbol Device:R_US
- added RV1, RV4: 100k, SynthStuff:Potentiometer_Alpha_RD901F-40-00D_Single_Vertical, symbol Device:R_Potentiometer_US
- added RV2, RV3, RV5, RV6: 100k, SynthStuff:Potentiometer_TT_P110KH1, symbol Device:R_Potentiometer_US
Connections:
- new net: J200.9 (Pin_9), J5.TN
- new net: J2.TN, J200.2 (Pin_2)
- new net: J200.8 (Pin_8), J6.TN
- new net: J1.TN, J200.1 (Pin_1)
- new net: J200.7 (Pin_7), J7.TN
- new net: R40.1, RV4.3
- new net: J200.6 (Pin_6), J8.TN
- new net: J200.3 (Pin_3), J3.TN
- new net: J200.4 (Pin_4), J4.TN
- new net: R21.1, RV1.3
- new net +12V: J50.1 (Pin_1), J60.1 (Pin_1), R21.2, R40.2
- new net CV 1 A Jack: J3.T, RV2.3
- new net CV 1 A Pot: J50.3 (Pin_3), RV2.2
- new net CV 1 B Jack: J7.T, RV5.3
- new net CV 1 B Pot: J60.3 (Pin_3), RV5.2
- new net CV 2 A Jack: J4.T, RV3.3
- new net CV 2 A Pot: J50.4 (Pin_4), RV3.2
- new net CV 2 B Jack: J8.T, RV6.3
- new net CV 2 B Pot: J60.4 (Pin_4), RV6.2
- new net GND: J0.1 (Pin_1), J1.S, J2.S, J200.10 (Pin_10), J200.5 (Pin_5), J3.S, J4.S, J5.S, J50.5 (Pin_5), J50.6 (Pin_6), J6.S, J60.5 (Pin_5), J60.6 (Pin_6), J7.S, J8.S, RV1.1, RV2.1, RV3.1, RV4.1, RV5.1, RV6.1
- new net Input A Jack: J1.T
- new net Input B Jack: J5.T
- new net Offset A Pot: J50.2 (Pin_2), RV1.2
- new net Offset B Pot: J60.2 (Pin_2), RV4.2
- new net Output A Jack: J2.T
- new net Output B Jack: J6.T
Other:
- note added: "Pots PCB"

Commit message: Finished Pots PCB
Parts:
- J50, J60: value Conn_01x06 -> Conn_01x08; footprint Connector_PinHeader_2.54mm:PinHeader_1x06_P2.54mm_Vertical -> Connector_PinHeader_2.54mm:PinHeader_1x08_P2.54mm_Vertical; symbol Connector_Generic:Conn_01x06 -> Connector_Generic:Conn_01x08
Connections:
- net +12V: now also J50.3 (Pin_3), J60.3 (Pin_3); no longer J50.1 (Pin_1), J60.1 (Pin_1)
- net CV 1 A Jack: now also J50.1 (Pin_1)
- net CV 1 A Pot: now also J50.5 (Pin_5); no longer J50.3 (Pin_3)
- net CV 1 B Jack: now also J60.1 (Pin_1)
- net CV 1 B Pot: now also J60.5 (Pin_5); no longer J60.3 (Pin_3)
- net CV 2 A Jack: now also J50.2 (Pin_2)
- net CV 2 A Pot: now also J50.6 (Pin_6); no longer J50.4 (Pin_4)
- net CV 2 B Jack: now also J60.2 (Pin_2)
- net CV 2 B Pot: now also J60.6 (Pin_6); no longer J60.4 (Pin_4)
- net GND: now also J50.7 (Pin_7), J50.8 (Pin_8), J60.7 (Pin_7), J60.8 (Pin_8); no longer J50.5 (Pin_5), J50.6 (Pin_6), J60.5 (Pin_5), J60.6 (Pin_6)
- net Offset A Pot: now also J50.4 (Pin_4); no longer J50.2 (Pin_2)
- net Offset B Pot: now also J60.4 (Pin_4); no longer J60.2 (Pin_2)

Commit message: Perfected pots (_conn) PCB
Parts:
- J0: now not fitted; now left out of the parts list
Changed lines of the file:
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@@
 		(unit 1)
 		(exclude_from_sim no)
-		(in_bom yes)
+		(in_bom no)
 		(on_board yes)
-		(dnp no)
+		(dnp yes)
 		(property "Reference" "J0"
 			(at 33.02 260.35 90)
